File: core/PCB/Wilssen_core_v0.201a.brd (EAGLE design)
At the start: 25.4 x 64.8 mm, 29 parts, among them Q1 8Mhz, U1 MAX1555, U2 3.3V, U3 ATMEGA168/ATMEGA328, X1 USBSMD

Commit message: 2.5V voltage reference + tidy up
Parts:
- removed R9: 1k, SparkFun:0402-RES
- added CC_TEXT1: CREATIVE_COMMONS, SparkFun-Aesthetics:CREATIVE_COMMONS
- added LOGO1: OSHW-LOGOS, SparkFun-Aesthetics:OSHW-LOGO-S
- added R6: 1k, rcl:R0805
- C10, C9: device SparkFun:0402-CAP -> SparkFun:0805
- R1: device SparkFun:0805 -> rcl:R0805
- R4: device SparkFun:1206 -> rcl:R0805
- moved JP4 9.61 mm to (10.2, 3.81), turned to 0 degrees
- moved U$1 8.82 mm to (12.7, 12.1), turned to 90 degrees
- moved C4 8.28 mm to (21.0, 1.91), turned to 270 degrees
- moved D1 5.08 mm to (7.62, 1.27)
- moved R1 3.18 mm to (6.35, 3.81)
- moved R3 3.18 mm to (15.9, 38.7)
- moved R2 3.18 mm to (12.7, 1.27)
- moved R4 1.42 mm to (17.8, 12.1)
Connections:
- net N$11: now also R6.2; no longer R9.1
- net N$8: now also R6.1; no longer R9.2
Routing:
- net A6: track 19.0 -> 2.12 mm, vias 2 -> 0
- net SCK: track 16.6 -> 2.37 mm
- net A7: track 16.0 -> 2.11 mm, vias 2 -> 0
- net VCC: track 24.5 -> 15.7 mm
- net N$1: track 5.98 -> 0.00 mm
- net RST: track 9.64 -> 3.93 mm
- net MISO: track 24.6 -> 20.8 mm
- net N$2: track 2.79 -> 0.00 mm
