File: core/PCB/Wilssen_core_v0.201a.sch (EAGLE design)
At the start: 29 parts, among them Q1 8Mhz, U1 MAX1555, U2 3.3V, U3 ATMEGA168/ATMEGA328, X1 USBSMD

Commit message: 2.5V voltage reference + tidy up
Parts:
- removed R9: 1k, SparkFun:RESISTOR0402-RES
- added CC_TEXT1: CREATIVE_COMMONS, SparkFun-Aesthetics:CREATIVE_COMMONS
- added LOGO1: OSHW-LOGOS, SparkFun-Aesthetics:OSHW-LOGOS
- added R6: 1k, rcl:R-EU_R0805
- C10, C9: device SparkFun:CAP0402-CAP -> SparkFun:CAP0805
- R1: device SparkFun:RESISTOR -> rcl:R-EU_R0805
- R4: device SparkFun:RESISTOR1206 -> rcl:R-EU_R0805
Connections:
- net N$11: now also R6.2; no longer R9.1
- net N$8: now also R6.1; no longer R9.2
Other:
- note added: "1"
- note added: "Wilssen core module"
- note added: "miniUSB socket"
- note removed: "Alex Shure"
- moved on the sheet: ATMEGA168/ATMEGA328, C5, C6, D1, JP1, JP2, JP3, JP8, JP9, Q1, U$1, U3
